File: pcb_v2/robot.sch (KiCad schematic (older format))
At the start: 23 parts, among them J1 M1 PWR, J11 MB CTRL, J12 MA CTRL, J2 M2 PWR, J3 Power Connector, J4 BATT, J5 TB6612_Motor_Driver, J7 PWR, Q1 2N3904, Q2 2N3904, U2 L7805, U3 L78L33_TO92

Commit message: SMB, 10 Dec 19, updated 3d print files.
Parts:
- added D2: LED, LED_THT:LED_D3.0mm, symbol Device:LED
- added Q3: 2N3906, Package_TO_SOT_THT:TO-92_Inline_Wide, symbol Transistor_BJT:2N3906
- added R2: 10k, Resistor_THT:R_Axial_DIN0207_L6.3mm_D2.5mm_P10.16mm_Horizontal, symbol Device:R
- added R7: 13k, Resistor_THT:R_Axial_DIN0207_L6.3mm_D2.5mm_P10.16mm_Horizontal, symbol Device:R
- added R8: 1k, Resistor_THT:R_Axial_DIN0207_L6.3mm_D2.5mm_P10.16mm_Horizontal, symbol Device:R
Connections:
- net +5V: now also Q3.1 (E)
- net +BATT: now also R2.1
- net GND: now also D2.1 (K), R7.2
- new net: Q3.2 (B), R2.2, R7.1
- new net: Q3.3 (C), R8.1
- new net: D2.2 (A), R8.2
Changed lines of the file:
@@
 Wire Wire Line
 	2800 1600 3150 1600
+$Comp
+L power:+BATT #PWR08
+U 1 1 5D3939F3
+P 3250 3800
+F 0 "#PWR08" H 3250 3650 50  0001 C CNN
+F 1 "+BATT" H 3265 3973 50  0000 C CNN
+F 2 "" H 3250 3800 50  0001 C CNN
+F 3 "" H 3250 3800 50  0001 C CNN
+	1    3250 3800
+	1    0    0    -1
+$EndComp
+$Comp
+L Device:R R2
+U 1 1 5D3A3C67
+P 3250 3950
+F 0 "R2" H 3320 3996 50  0000 L CNN
+F 1 "10k" H 3320 3905 50  0000 L CNN
+F 2 "Resistor_THT:R_Axial_DIN0207_L6.3mm_D2.5mm_P10.16mm_Horizontal" V 3180 3950 50  0001 C CNN
+F 3 "~" H 3250 3950 50  0001 C CNN
+	1    3250 3950
+	1    0    0    -1
+$EndComp
+$Comp
+L Device:R R7
+U 1 1 5D3A64D2
+P 3250 4250
+F 0 "R7" H 3320 4296 50  0000 L CNN
+F 1 "13k" H 3320 4205 50  0000 L CNN
+F 2 "Resistor_THT:R_Axial_DIN0207_L6.3mm_D2.5mm_P10.16mm_Horizontal" V 3180 4250 50  0001 C CNN
+F 3 "~" H 3250 4250 50  0001 C CNN
+	1    3250 4250
+	1    0    0    -1
+$EndComp
+$Comp
+L power:GND #PWR09
+U 1 1 5D3AA81B
+P 3250 4400
+F 0 "#PWR09" H 3250 4150 50  0001 C CNN
+F 1 "GND" H 3255 4227 50  0000 C CNN
+F 2 "" H 3250 4400 50  0001 C CNN
+F 3 "" H 3250 4400 50  0001 C CNN
+	1    3250 4400
+	1    0    0    -1
+$EndComp
+$Comp
+L Transistor_BJT:2N3906 Q3
+U 1 1 5D3AE71B
+P 2650 4100
+F 0 "Q3" H 2841 4054 50  0000 L CNN
+F 1 "2N3906" H 2841 4145 50  0000 L CNN
+F 2 "Package_TO_SOT_THT:TO-92_Inline_Wide" H 2850 4025 50  0001 L CIN
+F 3 "https://www.fairchildsemi.com/datasheets/2N/2N3906.pdf" H 2650 4100 50  0001 L CNN
+	1    2650 4100
+	-1   0    0    1
+$EndComp
+Wire Wire Line
+	2850 4100 3250 4100
+Connection ~ 3250 4100
+$Comp
+L power:+5V #PWR027
+U 1 1 5D3B3F50
+P 2550 3800
+F 0 "#PWR027" H 2550 3650 50  0001 C CNN
+F 1 "+5V" H 2565 3973 50  0000 C CNN
+F 2 "" H 2550 3800 50  0001 C CNN
+F 3 "" H 2550 3800 50  0001 C CNN
+	1    2550 3800
+	1    0    0    -1
+$EndComp
+Wire Wire Line
+	2550 3800 2550 3900
+$Comp
+L Device:R R8
+U 1 1 5D3B86CA
+P 2550 4450
+F 0 "R8" H 2620 4496 50  0000 L CNN
+F 1 "1k" H 2620 4405 50  0000 L CNN
+F 2 "Resistor_THT:R_Axial_DIN0207_L6.3mm_D2.5mm_P10.16mm_Horizontal" V 2480 4450 50  0001 C CNN
+F 3 "~" H 2550 4450 50  0001 C CNN
+	1    2550 4450
+	1    0    0    -1
+$EndComp
+$Comp
+L Device:LED D2
+U 1 1 5D3B8FAB
+P 2550 4750
+F 0 "D2" V 2589 4633 50  0000 R CNN
+F 1 "LED" V 2498 4633 50  0000 R CNN
+F 2 "LED_THT:LED_D3.0mm" H 2550 4750 50  0001 C CNN
+F 3 "~" H 2550 4750 50  0001 C CNN
+	1    2550 4750
+	0    -1   -1   0
+$EndComp
+$Comp
+L power:GND #PWR028
+U 1 1 5D3B9E7D
+P 2550 4900
+F 0 "#PWR028" H 2550 4650 50  0001 C CNN
+F 1 "GND" H 2555 4727 50  0000 C CNN
+F 2 "" H 2550 4900 50  0001 C CNN
+F 3 "" H 2550 4900 50  0001 C CNN
+	1    2550 4900
+	1    0    0    -1
+$EndComp
 $EndSCHEMATC
