File: pcb/pcb_v3/robot.sch (KiCad schematic (older format))
At the start: 28 parts, among them J1 M1 PWR, J11 MB CTRL, J12 MA CTRL, J2 M2 PWR, J3 Power Connector, J4 BATT, J5 TB6612_Motor_Driver, J7 SWITCH, Q1 2N3904, Q2 2N3904, Q3 2N3906, U1 L7805, U3 L78L33

Commit message: SMB, 29 Apr 2020, Updated a few things in PCB .
Parts:
- renumbered J7 to J1, J4 to J2, J12 to J3, J11 to J4, J1 to J5, J2 to J6, J3 to J7, J5 to J8, U3 to U2
Connections:
- net A2: no longer J3.2 (Pin_2), R6.1
- new net: J3.2 (Pin_2), R6.1
Other:
- note added: "Battery Indicator Circuit"
- moved on the sheet: C1, C2, C3, C4, C5, D1, D2, J1, J2, J3, J4, J5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
